Commit message: changed some much

File: robot_arm/urdf/rca.urdf (robot description, URDF)
Before this commit: robot ros_controlled_arm, 2 links, 1 joints
Links:
- link base_link: geometry collision cylinder length=0.058 radius=0.1; visual mesh filename=package://robot_arm/meshes/ scale=1.0

Commit message: working on a urdf. dont know why the stls not work

File: robot_arm/urdf/rca.urdf (robot description, URDF)
Before this commit: robot ros_controlled_arm, 2 links, 1 joints
Links:
- added link anker1, mass 10.0; collision box size=0.5 0.1 0.02; visual box size=0.5 0.03 0.02
- added link anker2, mass 10.0; collision box size=0.8 0.2 0.02; visual box size=0.5 0.03 0.02
- added link arm1_to_base, mass 10.0; collision cylinder length=0.058 radius=0.1; visual cylinder length=0.058 radius=0.1
- added link arm1_wurfel, mass 1.0; collision box size=0.04 0.09 0.06; visual box size=0.04 0.1 0.08
- added link arm2_to_wurfel, mass 1.0; collision box size=0.09 0.09 0.06; visual box size=0.03 0.5 0.08
- link base_link: geometry collision cylinder length=0.058 radius=0.1; visual cylinder length=0.058 radius=0.1
Joints:
- added joint anker2_to_base: type fixed, parent world, child anker2, origin xyz=0 0 0.01 rpy=0 0 1.57 , axis 0 0 0
- added joint anker_to_base: type fixed, parent world, child anker1, origin xyz=0 0 0.01 rpy=0 0 0, axis 0 0 0
- added joint arm2_to_arm1: type revolut, parent arm1_wurfel, child arm2_to_wurfel, origin xyz=-0.035 -0.23 0.02 rpy=0 0 0, axis 0 0 0
- added joint arm_base: type continuous, parent base_link, child arm1_to_base, origin xyz=0 0 0.0585 rpy=0 0 0, axis 0 0 0
- added joint wurfel_to_arm_base: type fixed, parent arm1_to_base, child arm1_wurfel, origin xyz=0 0.035 0.059 rpy=0 0 0, axis 0 0 0
